File: PCB/Secuenciador.kicad_pcb (KiCad board)
At the start: 2 copper layers, 7 parts, among them J1 JACK_ST_3SW_PROPER, U1 4050

Commit message: Rev 1.0
Parts:
- added 3.5mm_Screw: VAL**, 3.5mm_Screw, F.Cu at (114.2, 34.6)
- added 3.5mm_Screw: VAL**, 3.5mm_Screw, F.Cu at (114.2, 154.6)
- added 3.5mm_Screw: VAL**, 3.5mm_Screw, F.Cu at (34.2, 161.6)
- added BTNPAD1: ADAFRUIT_TRELLIS, Adafruit_trellis, F.Cu at (76.7, 115.3)
- added C1: CP1, C2V8, B.Cu at (35.8, 52.6)
- added C10: CP1, C2V10, B.Cu at (50.2, 91.6)
- added C11: C, C1, B.Cu at (34.8, 90.1)
- added C12: C, C1, B.Cu at (34.8, 87.1)
- added C13: C, C1, B.Cu at (55.8, 142.1)
- added C2: C, C1, B.Cu at (35.2, 59.1)
- added C3: C, C1, B.Cu at (35.2, 62.1)
- added C4: CP1, C2V8, B.Cu at (35.8, 80.6)
- added C5: C, C1, B.Cu at (56.8, 157.1)
- added C6: C, C1, B.Cu at (56.8, 160.1)
- added C7: CP1, C2V10, B.Cu at (63.8, 91.6)
- added C8: C, C1, B.Cu at (56.8, 107.6)
- added C9: C, C1, B.Cu at (53.8, 107.6)
- added CON1: BARREL_JACK, JACK_ALIM, B.Cu at (38.2, 37.1)
- added D1: DIODE, D3, B.Cu at (64.2, 63.1)
- added IC1: CNY17-3, DIP-6__300_ELL, B.Cu at (63.2, 54.6)
- added JP1: JUMPER, PIN_ARRAY_2X1, B.Cu at (56.2, 113.1)
- added JP2: JUMPER, PIN_ARRAY_2X1, B.Cu at (56.2, 130.6)
- added JP3: JUMPER, PIN_ARRAY_2X1, B.Cu at (56.8, 154.1)
- added JP4: JUMPER, PIN_ARRAY_2X1, B.Cu at (55.8, 147.6)
- added MIC1: MIC, PIN_ARRAY_3X1, F.Cu at (111.2, 160.6)
- added P1: DIN_5, MIDI_CONN, B.Cu at (58.2, 42.1)
- added P2: DIN_5, MIDI_CONN, B.Cu at (83.2, 42.1)
- added P3: PROGRAMMER, PINHEAD1-6, B.Cu at (40.8, 101.1)
- added R1: 10k, R1, B.Cu at (107.2, 67.1)
- added R2: 10k, R1, B.Cu at (107.2, 70.6)
- added R3: 10k, R1, B.Cu at (107.8, 60.6)
- added R4: 10k, R1, B.Cu at (104.2, 60.6)
- added R5: 10k, R1, B.Cu at (96.7, 91.6)
- added R6: 10k, R1, B.Cu at (99.7, 91.1)
- added R7: R, R1, B.Cu at (56.6, 53.9)
- added R8: R, R1, B.Cu at (53.8, 54.1)
- added R9: R, R1, B.Cu at (104.4, 54.7)
- added RV1: POT, PIN_ARRAY_3X1, F.Cu at (107.2, 88.6)
- J1: value JACK_ST_3SW_PROPER -> JACK_ST_2SW_PROPER; footprint Jack_6.35_Stereo_SW -> Jack_3.5mm_Stereo
- LCD1: footprint pin_array_8x2 -> Nokia5110_LCD_2
- MCU1: value PRO_MINI_2 -> MAPLE_MINI; footprint ProMiniThick -> Leaf_maple_mini; moved to B.Cu
- MP31: moved to B.Cu
- U1: value 4050 -> 7805; footprint DIP-16__300_ELL -> TO220_VERT; moved to B.Cu
- moved MCU1 146.7 mm to (49.8, 157.6), turned to 90 degrees
- moved MP31 120.4 mm to (103.2, 159.6), turned to 90 degrees
- moved ENC2 91.6 mm to (93.2, 84.1), turned to 180 degrees
- moved ENC1 75.1 mm to (93.2, 52.1)
- moved J1 61.5 mm to (105.2, 38.6)
- moved U1 20.1 mm to (35.2, 69.6), turned to 180 degrees
- moved LCD1 16.0 mm to (53.2, 41.1)
Connections:
- ENC1 pad 1: (no net) -> GND
- ENC1 pad 2: (no net) -> /ENC1_L1
- ENC1 pad 3: (no net) -> /ENC1_L2
- ENC1 pad 4: (no net) -> /ENC1_SW
- ENC1 pad 5: (no net) -> /ENC1_A
- ENC1 pad 6: (no net) -> GND
- ENC1 pad 7: (no net) -> /ENC1_B
- ENC2 pad 1: (no net) -> GND
- ENC2 pad 2: (no net) -> /ENC2_L1
- ENC2 pad 4: (no net) -> /ENC2_SW
- ENC2 pad 5: (no net) -> /ENC2_A
- ENC2 pad 6: (no net) -> GND
- ENC2 pad 7: (no net) -> /ENC2_B
- LCD1 pad 7: +5V -> /DISP_LED
- MCU1 pad 1: (no net) -> +3.3V
- MCU1 pad 10: (no net) -> /VS1053_SDCS
- MCU1 pad 11: (no net) -> /VS1053_XDCS
- MCU1 pad 12: /VS1053_RST -> /VS1053_CS
- MCU1 pad 13: /SCL -> /VS1053_SCLK
- MCU1 pad 14: /SDA -> /VS1053_MISO
- MCU1 pad 15: (no net) -> /VS1053_MOSI
- MCU1 pad 16: (no net) -> /VS1053_DREQ
- MCU1 pad 17: (no net) -> /Boot1
- MCU1 pad 18: /MOSI_5V -> /MIDI_OUT
- MCU1 pad 19: (no net) -> /MIDI_IN
- MCU1 pad 2: (no net) -> AGND
- MCU1 pad 20: /SCLK_3V3 -> +5V
- MCU1 pad 21: (no net) -> /CS_3V3
- MCU1 pad 22: (no net) -> /SCLK_3V3
- MCU1 pad 24: (no net) -> /MOSI_3V3
- MCU1 pad 26: (no net) -> /PROG_TX
- MCU1 pad 27: GND -> /PROG_RX
- MCU1 pad 4: GND -> /ENC1_A
- MCU1 pad 5: /VS1053_RX -> /ENC1_SW
- MCU1 pad 6: /RST_5V -> /ENC2_A
- MCU1 pad 7: /CS_3V3 -> N-0000039
- MCU1 pad 8: /DC_5V -> /DC_3V3
- MCU1 pad 9: (no net) -> /RST_3V3
- MP31 pad 15: /VS1053_RX -> /MIDI_OUT
- MP31 pad 17: (no net) -> /VS1053_XDCS
- MP31 pad 18: (no net) -> /VS1053_SDCS
- MP31 pad 19: (no net) -> /VS1053_CS
- MP31 pad 2: (no net) -> /MIC+
- MP31 pad 21: (no net) -> /VS1053_SCLK
- MP31 pad 22: (no net) -> /VS1053_MOSI
- MP31 pad 23: (no net) -> /VS1053_MISO
- MP31 pad 25: +3.3V -> (no net)
- MP31 pad 27: (no net) -> /VS1053_DREQ
- MP31 pad 3: (no net) -> AGND
- MP31 pad 4: (no net) -> AGND
- MP31 pad 7: +3.3V -> N-0000028
Routing:
- net +5V: track 0.00 -> 317.9 mm, vias 0 -> 2
- net AGND: track 0.00 -> 218.8 mm, vias 0 -> 1
- net /ENC2_A: track 0.00 -> 159.0 mm, vias 0 -> 2
- net +3.3V: track 0.00 -> 143.8 mm
- net /ENC1_A: track 0.00 -> 143.7 mm, vias 0 -> 2
- net /ENC1_SW: track 0.00 -> 138.9 mm, vias 0 -> 2
- net /MIDI_OUT: track 0.00 -> 138.9 mm, vias 0 -> 1
- net /ENC1_L1: track 0.00 -> 117.2 mm, vias 0 -> 2
- net /SCL: track 0.00 -> 112.4 mm, vias 0 -> 3
- net /SDA: track 0.00 -> 110.7 mm, vias 0 -> 2
- net /ENC1_L2: track 0.00 -> 108.7 mm, vias 0 -> 5
- net /LOUT: track 0.00 -> 105.7 mm
- net /ROUT: track 0.00 -> 101.6 mm
- net /ENC2_SW: track 0.00 -> 88.9 mm, vias 0 -> 2
- net /ENC2_L1: track 0.00 -> 87.5 mm, vias 0 -> 2
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- added copper zone on B.Cu, net GND
Other:
- board outline added: 87.5 x 135 mm
- net class Speed added: clearance 0.254, trace_width 0.2032, via_dia 0.889, via_drill 0.635
- net class Supply added: clearance 0.254, trace_width 0.3048, via_dia 0.889, via_drill 0.635
- rule trace_min: 0.254 -> 0.2032
- board text added: "Boot1->GND"
- board text added: "DTR"
- board text added: "HACKERSPACE CHOLULA"
- board text added: "P1->3V3"
- board text added: "REV 1.0"
- board text added: "SECUENCIADOR MIDI"
- board text added: "VS1053 Reset"
